File: rocket2-battery.kicad_sch (KiCad schematic)
At the start: 55 parts, among them J1 Conn_01x07, J2 SMA, J3 ARM Cortex Debug, P1 PAD_SMD, P2 PAD_SMD, P3 PAD_SMD, P4 PAD_SMD, Q1 NMOS, Q2 NMOS, Q3 PMOS, Q4 PMOS, Q5 NMOS, Q6 NMOS, Q7 PMOS, Q8 PMOS, Y1 16MHz

Commit message: Fixed issues
Parts:
- added P5, P6, P7: PAD_SMD, TestPoint:TestPoint_Pad_2.0x2.0mm, symbol pkl_misc:PAD_SMD
- C1, C3: Manufacturer Generic -> Samsung; Part # (none) -> CL10B105KL9VPNC
- D1: Part # (none) -> Generic 0603 Green LED
- J1: Part # (none) -> Generic 2.54mm 1x7 Pin Header
- R1: Part # (none) -> Generic 0603 3.3K 5% Resistor
- R10: renamed from R9; value 1.5k -> 15K; Part # (none) -> Generic 0603 15K 0.1% Resistor
- R11: renamed from R10; Part # (none) -> Generic 0603 100ohm 5% Resistor
- R12, R5: value 10k -> 10K; Part # (none) -> Generic 0603 10K 1% Resistor
- R13, R6: Part # (none) -> Generic 0603 100ohm 5% Resistor
- R14, R7: value 10k -> 100k; Part # (none) -> Generic 0603 100K 0.1% Resistor
- R15: value 1.5k -> 15K; Part # (none) -> Generic 0603 15K 0.1% Resistor
- R2: renamed from R4; value 1k -> 1K; Part # (none) -> Generic 0603 1K 10% Resistor
- R4: renamed from R2; Part # (none) -> Generic 0603 100ohm 5% Resistor
- R9: renamed from R11; value 1k -> 1K; Part # (none) -> Generic 0603 1K 10% Resistor
Connections:
- net BAT_OUT+: no longer C1.1, Q7.3 (S), Q8.3 (S), R12.1, R14.1, U1.1 (IN)
- net GND: now also P6.1 (PAD)
- net MAIN+: now also P7.1 (PAD)
- net MOSFET1: now also R2.2
- net MOSFET2: now also R9.2
- net at Q5.2 (G), Q6.2 (G), R11.2: no longer R9.2
- net at Q1.2 (G), Q2.2 (G), R4.2: no longer R2.2
- new net BATT_MAIN+: C1.1, P5.1 (PAD), Q7.3 (S), Q8.3 (S), R12.1, R14.1, U1.1 (IN)
Other:
- moved on the sheet: R2, R4, R9
